File: andrew_badge/andrew_badge.kicad_pcb (KiCad board)
At the start: 2 copper layers, 71.5 x 88 mm, 16 parts, among them SW1 SW_Push, SW2 SW_Push, SW3 SW_Push, U1 CC1101_module, U2 ESP32-C3_SUPERMINI_TH, U3 ER_OLEDM0.91_1x-I2C, U4 3*AAA_holder

Commit message: added power switch
Parts:
- added SW5: SW_SPDT, Button_Switch_THT:SW_Slide_SPDT_Angled_CK_OS102011MA1Q, F.Cu at (136.5, 69.5)
Connections:
- U4 pad 1: pack+ -> Net-(SW5-C)
Routing:
- net pack+: track 55.6 -> 34.1 mm
- net Net-(SW5-C): track 0.00 -> 20.0 mm
Other:
- board text added: "ABER"
- board text added: "Built for Fallout Shenzhen, July '26"
- board text added: "DA"
- board text added: "IMMER"
- board text added: "NOCH"
- board text added: "SIND"
- board text added: "WIR"
